Commit message: moveit + control

File: src/ur5e_robotiq_moveit_config/srdf/ur.srdf.xacro (robot description, xacro)
@@ -1,12 +1,20 @@
 <?xml version="1.0" encoding="UTF-8"?>
-<robot xmlns:xacro="http://wiki.ros.org/xacro" name="$(arg name)">
+<robot xmlns:xacro="http://www.ros.org/wiki/xacro" name="ur">
   <!-- robot name parameter -->
-  <xacro:arg name="name" default="ur"/>
+  <xacro:arg name="name" default="ur5e"/>
   <xacro:include filename="$(find ur_moveit_config)/srdf/ur_macro.srdf.xacro"/>
   <xacro:ur_srdf/>
-  <group name="gripper">
-    <joint name="rq_robotiq_85_left_knuckle_joint"/>
-    <joint name="rq_robotiq_85_right_knuckle_joint"/>
-  </group>
-  <end_effector name="robotiq_2f85" parent_link="tool0" group="gripper"/>
+    <!-- Robotiq: allow self-collisions for adjacent/mimic links -->
+  <disable_collisions link1="rq_robotiq_85_base_link" link2="rq_robotiq_85_left_knuckle_link" reason="Adjacent"/>
+  <disable_collisions link1="rq_robotiq_85_base_link" link2="rq_robotiq_85_left_inner_knuckle_link" reason="Adjacent"/>
+  <disable_collisions link1="rq_robotiq_85_base_link" link2="rq_robotiq_85_right_knuckle_link" reason="Adjacent"/>
+  <disable_collisions link1="rq_robotiq_85_base_link" link2="rq_robotiq_85_right_inner_knuckle_link" reason="Adjacent"/>
+  <disable_collisions link1="rq_robotiq_85_left_finger_link" link2="rq_robotiq_85_left_finger_tip_link" reason="Adjacent"/>
+  <disable_collisions link1="rq_robotiq_85_right_finger_link" link2="rq_robotiq_85_right_finger_tip_link" reason="Adjacent"/>
+  <disable_collisions link1="rq_robotiq_85_left_finger_link" link2="rq_robotiq_85_left_knuckle_link" reason="Adjacent"/>
+  <disable_collisions link1="rq_robotiq_85_left_finger_tip_link" link2="rq_robotiq_85_left_inner_knuckle_link" reason="Adjacent"/>
+  <disable_collisions link1="rq_robotiq_85_right_finger_link" link2="rq_robotiq_85_right_knuckle_link" reason="Adjacent"/>
+  <disable_collisions link1="rq_robotiq_85_right_finger_tip_link" link2="rq_robotiq_85_right_inner_knuckle_link" reason="Adjacent"/>
+  <!-- If your mounting causes contact at zero, allow it -->
+  <disable_collisions link1="rq_robotiq_85_base_link" link2="wrist_3_link" reason="NeverCollide"/>
 </robot>

File: src/ur5e_robotiq_moveit_config/srdf/ur_macro.srdf.xacro (robot description, xacro)
@@ -1,18 +1,19 @@
 <?xml version="1.0" encoding="UTF-8"?>
 <robot xmlns:xacro="http://wiki.ros.org/xacro">
-<!--This does not replace URDF, and is not an extension of URDF.
-    This is a format for representing semantic information about the robot structure.
-    A URDF file must exist for this robot as well, where the joints and the links that are referenced are defined
--->
+  <!--
+    SRDF (Semantic Robot Description Format) macro used by UR MoveIt config.
+    This defines planning groups, named states, end effectors, and disabled collisions.
+  -->
   <xacro:macro name="ur_srdf" params="">
-    <!--GROUPS - Representation of a set of joints and links. This can be useful for specifying DOF to plan for, defining arms, end effectors, etc-->
-    <!--LINKS - When a link is specified, the parent joint of that link (if it exists) is automatically included-->
-    <!--JOINTS - When a joint is specified, the child link of that joint (which will always exist) is automatically included-->
-    <!--CHAINS - When a chain is specified, all the links along the chain (including endpoints) are included in the group. Additionally, all the joints that are parents to included links are also included. This means that joints along the chain and the parent joint of the base link are included in the group-->
-    <!--SUBGROUPS - Groups can also be formed by referencing to already defined group names-->
+    <!-- ======================= GROUPS ======================= -->
     <group name="ur_manipulator">
       <chain base_link="base_link" tip_link="tool0" />
     </group>
-    <!--GROUP STATES - Purpose - Define a named state for a particular group, in terms of joint values. This is useful to define states like 'folded arms'-->
+    <!-- Robotiq 2F-85 gripper group (from ur_yt_sim URDF joint list) -->
+    <group name="robotiq_gripper">
+      <!-- Primary actuated joint for this Robotiq URDF -->
+      <joint name="rq_robotiq_85_left_knuckle_joint" />
+    </group>
+    <!-- ===================== GROUP STATES ==================== -->
     <group_state name="home" group="ur_manipulator">
       <joint name="elbow_joint" value="0" />
@@ -39,7 +40,11 @@
       <joint name="wrist_3_joint" value="-0.11" />
     </group_state>
-    <!--END EFFECTOR - Purpose - Represent information about an end effector.-->
-    <!--VIRTUAL JOINT - Purpose - this element defines a virtual joint between a robot link and an external frame of reference (considered fixed with respect to the robot)-->
-    <!--DISABLE COLLISIONS - By default it is assumed that any link of the robot could potentially come into collision with any other link in the robot. This tag disables collision checking between a specified pair of links. -->
+    <!-- ==================== END EFFECTOR ===================== -->
+    <!-- The gripper is attached to tool0 in your URDF/xacro. -->
+    <end_effector
+      name="robotiq_2f85"
+      parent_link="tool0"
+      group="robotiq_gripper" />
+    <!-- ================= DISABLE COLLISIONS ================== -->
     <disable_collisions link1="base_link" link2="base_link_inertia" reason="Adjacent" />
     <disable_collisions link1="base_link_inertia" link2="shoulder_link" reason="Adjacent" />

File: src/ur_yt_sim/urdf/ur5.ros2_control.xacro (robot description, xacro)
@@ -30,4 +30,5 @@
           <plugin>ign_ros2_control/IgnitionSystem</plugin>
         </xacro:if>
+        <!-- Route A (simulation / fake hardware) -->
         <xacro:if value="${use_fake_hardware}">
           <plugin>mock_components/GenericSystem</plugin>
@@ -36,4 +37,5 @@
           <param name="calculate_dynamics">true</param>
         </xacro:if>
+        <!-- Real hardware ONLY -->
         <xacro:unless value="${use_fake_hardware or sim_gazebo or sim_ignition}">
           <plugin>ur_robot_driver/URPositionHardwareInterface</plugin>
@@ -65,65 +67,57 @@
         </xacro:unless>
       </hardware>
+      <!-- ================= ARM JOINTS ONLY =================
+           IMPORTANT:
+           - Do NOT put any Robotiq joints here.
+           - Do NOT export GPIO/sensors in fake hardware.
+           - Keep command interface = position only (matches your controller config).
+      -->
       <joint name="${tf_prefix}shoulder_pan_joint">
         <command_interface name="position"/>
-        <command_interface name="velocity"/>
-        <state_interface name="position">
-          <!-- initial position for the FakeSystem and simulation -->
+        <state_interface name="position">
           <param name="initial_value">${initial_positions['shoulder_pan_joint']}</param>
         </state_interface>
         <state_interface name="velocity"/>
-        <state_interface name="effort"/>
       </joint>
       <joint name="${tf_prefix}shoulder_lift_joint">
         <command_interface name="position"/>
-        <command_interface name="velocity"/>
-        <state_interface name="position">
-          <!-- initial position for the FakeSystem and simulation -->
+        <state_interface name="position">
           <param name="initial_value">${initial_positions['shoulder_lift_joint']}</param>
         </state_interface>
         <state_interface name="velocity"/>
-        <state_interface name="effort"/>
       </joint>
       <joint name="${tf_prefix}elbow_joint">
         <command_interface name="position"/>
-        <command_interface name="velocity"/>
-        <state_interface name="position">
-          <!-- initial position for the FakeSystem and simulation -->
+        <state_interface name="position">
           <param name="initial_value">${initial_positions['elbow_joint']}</param>
         </state_interface>
         <state_interface name="velocity"/>
-        <state_interface name="effort"/>
       </joint>
       <joint name="${tf_prefix}wrist_1_joint">
         <command_interface name="position"/>
-        <command_interface name="velocity"/>
-        <state_interface name="position">
-          <!-- initial position for the FakeSystem and simulation -->
+        <state_interface name="position">
           <param name="initial_value">${initial_positions['wrist_1_joint']}</param>
         </state_interface>
         <state_interface name="velocity"/>
-        <state_interface name="effort"/>
       </joint>
       <joint name="${tf_prefix}wrist_2_joint">
         <command_interface name="position"/>
-        <command_interface name="velocity"/>
-        <state_interface name="position">
-          <!-- initial position for the FakeSystem and simulation -->
+        <state_interface name="position">
           <param name="initial_value">${initial_positions['wrist_2_joint']}</param>
         </state_interface>
         <state_interface name="velocity"/>
-        <state_interface name="effort"/>
       </joint>
       <joint name="${tf_prefix}wrist_3_joint">
         <command_interface name="position"/>
-        <command_interface name="velocity"/>
-        <state_interface name="position">
-          <!-- initial position for the FakeSystem and simulation -->
+        <state_interface name="position">
           <param name="initial_value">${initial_positions['wrist_3_joint']}</param>
         </state_interface>
         <state_interface name="velocity"/>
-        <state_interface name="effort"/>
-      </joint>
-      <xacro:unless value="${sim_gazebo or sim_ignition}">
+      </joint>
+      <!-- ================= REAL HW ONLY: sensors + GPIO =================
+           These interfaces are NOT exported by mock_components/GenericSystem.
+           So keep them ONLY for real hardware.
+      -->
+      <xacro:unless value="${use_fake_hardware or sim_gazebo or sim_ignition}">
         <sensor name="${tf_prefix}tcp_fts_sensor">
           <state_interface name="force.x"/>
@@ -143,5 +137,4 @@
           <state_interface name="orientation.w"/>
         </sensor>
-        <!-- NOTE The following are joints used only for testing with fake hardware and will change in the future -->
         <gpio name="${tf_prefix}speed_scaling">
           <state_interface name="speed_scaling_factor"/>
@@ -278,57 +271,57 @@
         </gpio>
         <gpio name="${tf_prefix}force_mode">
-        <command_interface name="task_frame_x"/>
-        <command_interface name="task_frame_y"/>
-        <command_interface name="task_frame_z"/>
-        <command_interface name="task_frame_rx"/>
-        <command_interface name="task_frame_ry"/>
-        <command_interface name="task_frame_rz"/>
-        <command_interface name="selection_vector_x"/>
-        <command_interface name="selection_vector_y"/>
-        <command_interface name="selection_vector_z"/>
-        <command_interface name="selection_vector_rx"/>
-        <command_interface name="selection_vector_ry"/>
-        <command_interface name="selection_vector_rz"/>
-        <command_interface name="wrench_x"/>
-        <command_interface name="wrench_y"/>
-        <command_interface name="wrench_z"/>
-        <command_interface name="wrench_rx"/>
-        <command_interface name="wrench_ry"/>
-        <command_interface name="wrench_rz"/>
-        <command_interface name="limits_x"/>
-        <command_interface name="limits_y"/>
-        <command_interface name="limits_z"/>
-        <command_interface name="limits_rx"/>
-        <command_interface name="limits_ry"/>
-        <command_interface name="limits_rz"/>
-        <command_interface name="type"/>
-        <command_interface name="damping"/>
-        <command_interface name="gain_scaling"/>
-        <command_interface name="disable_cmd"/>
-        <command_interface name="force_mode_async_success"/>
-      </gpio>
-      <gpio name="${tf_prefix}trajectory_passthrough">
-        <command_interface name="setpoint_positions_0"/>
-        <command_interface name="setpoint_positions_1"/>
-        <command_interface name="setpoint_positions_2"/>
-        <command_interface name="setpoint_positions_3"/>
-        <command_interface name="setpoint_positions_4"/>
-        <command_interface name="setpoint_positions_5"/>
-        <command_interface name="setpoint_velocities_0"/>
-        <command_interface name="setpoint_velocities_1"/>
-        <command_interface name="setpoint_velocities_2"/>
-        <command_interface name="setpoint_velocities_3"/>
-        <command_interface name="setpoint_velocities_4"/>
-        <command_interface name="setpoint_velocities_5"/>
-        <command_interface name="setpoint_accelerations_0"/>
-        <command_interface name="setpoint_accelerations_1"/>
-        <command_interface name="setpoint_accelerations_2"/>
-        <command_interface name="setpoint_accelerations_3"/>
-        <command_interface name="setpoint_accelerations_4"/>
-        <command_interface name="setpoint_accelerations_5"/>
-        <command_interface name="transfer_state"/>
-        <command_interface name="time_from_start"/>
-        <command_interface name="abort"/>
-      </gpio>
+          <command_interface name="task_frame_x"/>
+          <command_interface name="task_frame_y"/>
+          <command_interface name="task_frame_z"/>
+          <command_interface name="task_frame_rx"/>
+          <command_interface name="task_frame_ry"/>
+          <command_interface name="task_frame_rz"/>
+          <command_interface name="selection_vector_x"/>
+          <command_interface name="selection_vector_y"/>
+          <command_interface name="selection_vector_z"/>
+          <command_interface name="selection_vector_rx"/>
+          <command_interface name="selection_vector_ry"/>
+          <command_interface name="selection_vector_rz"/>
+          <command_interface name="wrench_x"/>
+          <command_interface name="wrench_y"/>
+          <command_interface name="wrench_z"/>
+          <command_interface name="wrench_rx"/>
+          <command_interface name="wrench_ry"/>
+          <command_interface name="wrench_rz"/>
+          <command_interface name="limits_x"/>
+          <command_interface name="limits_y"/>
+          <command_interface name="limits_z"/>
+          <command_interface name="limits_rx"/>
+          <command_interface name="limits_ry"/>
+          <command_interface name="limits_rz"/>
+          <command_interface name="type"/>
+          <command_interface name="damping"/>
+          <command_interface name="gain_scaling"/>
+          <command_interface name="disable_cmd"/>
+          <command_interface name="force_mode_async_success"/>
+        </gpio>
+        <gpio name="${tf_prefix}trajectory_passthrough">
+          <command_interface name="setpoint_positions_0"/>
+          <command_interface name="setpoint_positions_1"/>
+          <command_interface name="setpoint_positions_2"/>
+          <command_interface name="setpoint_positions_3"/>
+          <command_interface name="setpoint_positions_4"/>
+          <command_interface name="setpoint_positions_5"/>
+          <command_interface name="setpoint_velocities_0"/>
+          <command_interface name="setpoint_velocities_1"/>
+          <command_interface name="setpoint_velocities_2"/>
+          <command_interface name="setpoint_velocities_3"/>
+          <command_interface name="setpoint_velocities_4"/>
+          <command_interface name="setpoint_velocities_5"/>
+          <command_interface name="setpoint_accelerations_0"/>
+          <command_interface name="setpoint_accelerations_1"/>
+          <command_interface name="setpoint_accelerations_2"/>
+          <command_interface name="setpoint_accelerations_3"/>
+          <command_interface name="setpoint_accelerations_4"/>
+          <command_interface name="setpoint_accelerations_5"/>
+          <command_interface name="transfer_state"/>
+          <command_interface name="time_from_start"/>
+          <command_interface name="abort"/>
+        </gpio>
         <gpio name="${tf_prefix}get_robot_software_version">
           <state_interface name="get_version_major"/>

File: src/ur_yt_sim/urdf/ur_moveit.urdf.xacro (robot description, xacro)
@@ -1,13 +1,19 @@
 <?xml version="1.0"?>
 <robot xmlns:xacro="http://wiki.ros.org/xacro" name="ur">
-  <!-- xacro args MUST be declared before use -->
-  <xacro:arg name="name" default="ur"/>
+  <!-- ===================== ARGS ===================== -->
+  <xacro:arg name="name" default="ur5e"/>
   <xacro:arg name="ur_type" default="ur5e"/>
   <xacro:arg name="tf_prefix" default=""/>
-  <!-- Now it's safe to use $(arg name) -->
-  <xacro:property name="robot_name" value="$(arg name)"/>
+  <!-- Route A: fake ros2_control for arm + gripper -->
+  <xacro:arg name="use_fake_hardware" default="true"/>
+  <xacro:arg name="fake_sensor_commands" default="false"/>
+  <!-- ===================== INCLUDES ===================== -->
   <xacro:include filename="$(find ur_description)/urdf/ur_macro.xacro"/>
+  <!-- UR arm ros2_control macro (from your ur_yt_sim pkg) -->
+  <xacro:include filename="$(find ur_yt_sim)/urdf/ur5.ros2_control.xacro"/>
+  <!-- Robotiq: geometry macro + our ros2_control override macro -->
   <xacro:include filename="$(find robotiq_description)/urdf/robotiq_2f_85_macro.urdf.xacro"/>
-  <!-- params -->
+  <xacro:include filename="$(find ur_yt_sim)/urdf/robotiq_overrides/robotiq_gripper.ros2_control.xacro"/>
+  <!-- ===================== UR PARAM FILES ===================== -->
   <xacro:arg name="joint_limit_params"
              default="$(find ur_description)/config/$(arg ur_type)/joint_limits.yaml"/>
@@ -18,5 +24,7 @@
   <xacro:arg name="visual_params"
              default="$(find ur_description)/config/$(arg ur_type)/visual_parameters.yaml"/>
+  <!-- ===================== WORLD ===================== -->
   <link name="world"/>
+  <!-- ===================== UR ROBOT (geometry + joints) ===================== -->
   <xacro:ur_robot
     name="$(arg name)"
@@ -29,6 +37,38 @@
     <origin xyz="0 0 0" rpy="0 0 0"/>
   </xacro:ur_robot>
-  <xacro:robotiq_gripper name="robotiq_2f85" parent="tool0" prefix="rq_">
+  <!-- ===================== UR ARM ROS2_CONTROL (FAKE) ===================== -->
+  <!-- NOTE: This is what provides shoulder_pan_joint/position etc. -->
+  <xacro:ur_ros2_control
+    name="$(arg name)"
+    use_fake_hardware="$(arg use_fake_hardware)"
+    fake_sensor_commands="$(arg fake_sensor_commands)"
+    sim_gazebo="false"
+    sim_ignition="false"
+    headless_mode="true"
+    tf_prefix="$(arg tf_prefix)"
+    script_filename="/tmp/ur_fake.script"
+    output_recipe_filename="/tmp/ur_fake_out.recipe"
+    input_recipe_filename="/tmp/ur_fake_in.recipe"
+    hash_kinematics=""
+    robot_ip="0.0.0.0" />
+  <!-- ===================== ROBOTIQ GEOMETRY ONLY (NO ros2_control) ===================== -->
+  <xacro:robotiq_gripper
+    name="robotiq_2f85"
+    parent="tool0"
+    prefix="rq_"
+    include_ros2_control="false"
+    sim_ignition="false"
+    sim_isaac="false"
+    use_fake_hardware="$(arg use_fake_hardware)"
+    fake_sensor_commands="$(arg fake_sensor_commands)">
     <origin xyz="0 0 0" rpy="0 0 0"/>
   </xacro:robotiq_gripper>
+  <!-- ===================== ROBOTIQ ROS2_CONTROL (FAKE) ===================== -->
+  <xacro:robotiq_gripper_ros2_control
+    name="robotiq_2f85"
+    prefix="rq_"
+    sim_ignition="false"
+    sim_isaac="false"
+    use_fake_hardware="$(arg use_fake_hardware)"
+    fake_sensor_commands="$(arg fake_sensor_commands)"/>
 </robot>
